Commit message: upd sensor position

File: turtlebot3_parc/urdf/sensors.xacro (robot description, xacro)
@@ -6,5 +6,5 @@
   <!-- Realsense sensor -->
   <xacro:sensor_d435i parent="base_link" use_nominal_extrinsics="true">
-    <origin xyz="0.3 0 0.11" rpy="0 0 0" />
+    <origin xyz="0.0 0 0.11" rpy="0 0 0" />
   </xacro:sensor_d435i>
   <!-- Realsense Gazebo Plugin -->
